File: HalfBridge_GateDriver.kicad_sch (KiCad schematic)
At the start: 43 parts, among them SW1 CAS-D20X1, SW2 CAS-D20X1, U1 74AHC1G86, U2 74AHC1G86, U3 74AHC1G86, U4 RKD-052005D, U5 NCD57252, U6 RKD-052005D

Commit message: diff circuit
Parts:
- added C12, C4, C5, C6: 100n, Capacitor_SMD:C_0603_1608Metric_Pad1.08x0.95mm_HandSolder, symbol Device:C
- renumbered C7 to C10, C8 to C11, C9 to C13, C10 to C14, C11 to C15, C12 to C16, C13 to C17, C14 to C18, C15 to C19, C16 to C20, C17 to C21, C4 to C7, C5 to C8, C6 to C9
Connections:
- net dis: now also SW2.2 (B); no longer SW2.5 (B)
- net dis_i: now also SW2.1 (A), SW2.5 (B); no longer SW2.2 (B), SW2.6 (C)
- net dis_x: now also SW2.3 (C); no longer SW2.4 (A)
- net gnd: now also SW2.4 (A), C12.2, C4.2, C5.2, C6.2; no longer SW2.3 (C)
- net vcc: now also SW2.6 (C), C4.1, C5.1, C6.1; no longer SW2.1 (A)
- net vcci: now also C12.1
Other:
- moved on the sheet: U3
