File: HalfBridge_SiC.kicad_sch (KiCad schematic)
At the start: 4 parts, among them J4 Screw_Terminal_01x02, SW2 CAS-D20X1

Commit message: quad diff receiver
Other:
- sheet HalfBridge_GateDriver ports: added dis_x; removed none
Changed lines of the file:
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@@
-	(wire
-		(pts
-			(xy 53.34 100.33) (xy 102.87 100.33)
-		)
-		(stroke
-			(width 0)
-			(type default)
-		)
-	)
 	(wire
 		(pts
@@
 	(wire
 		(pts
-			(xy 54.61 102.87) (xy 102.87 102.87)
-		)
-		(stroke
-			(width 0)
-			(type default)
-		)
-	)
-	(wire
-		(pts
 			(xy 81.28 66.04) (xy 81.28 95.25)
 		)
@@
 	(wire
 		(pts
-			(xy 54.61 97.79) (xy 54.61 102.87)
-		)
-		(stroke
-			(width 0)
-			(type default)
-		)
-	)
-	(wire
-		(pts
 			(xy 83.82 82.55) (xy 82.55 82.55)
 		)
@@
 	(wire
 		(pts
+			(xy 54.61 105.41) (xy 54.61 97.79)
+		)
+		(stroke
+			(width 0)
+			(type default)
+		)
+	)
+	(wire
+		(pts
 			(xy 95.25 68.58) (xy 95.25 95.25)
 		)
@@
 	(wire
 		(pts
+			(xy 102.87 105.41) (xy 54.61 105.41)
+		)
+		(stroke
+			(width 0)
+			(type default)
+		)
+	)
+	(wire
+		(pts
+			(xy 102.87 102.87) (xy 53.34 102.87)
+		)
+		(stroke
+			(width 0)
+			(type default)
+		)
+	)
+	(wire
+		(pts
 			(xy 142.24 100.33) (xy 154.94 100.33)
 		)
@@
 	(wire
 		(pts
-			(xy 53.34 95.25) (xy 53.34 100.33)
+			(xy 53.34 102.87) (xy 53.34 95.25)
 		)
 		(stroke
@@
 	(sheet
 		(at 102.87 92.71)
-		(size 39.37 12.7)
+		(size 39.37 15.24)
 		(fields_autoplaced yes)
 		(stroke
@@
 		)
 		(property "Sheetfile" "HalfBridge_GateDriver.kicad_sch"
-			(at 102.87 105.9946 0)
+			(at 102.87 108.5346 0)
 			(effects
 				(font
@@
 		)
 		(pin "vcc" input
-			(at 102.87 100.33 180)
+			(at 102.87 102.87 180)
 			(effects
 				(font
@@
 		)
 		(pin "gnd" input
-			(at 102.87 102.87 180)
+			(at 102.87 105.41 180)
 			(effects
 				(font
@@
 			(effects
 				(font
+					(size 1.27 1.27)
+				)
+				(justify left)
+			)
+		)
+		(pin "dis_x" input
+			(at 102.87 100.33 180)
+			(effects
+				(font

Commit message: new optical diff xor
Parts:
- removed SW2: CAS-D20X1, My_Button_Switch_SMD:Nidec_Copal_CAS-D20A1, symbol My_Switch:CAS-D20X1
- renumbered D3 to D1, J4 to J1, R17 to R1
Other:
- sheet HalfBridge_GateDriver ports: added en; removed dis_x
- sheet HalfBridge_Optical ports: added inen; removed none
