File: HalfBridge_SiC.kicad_sch (KiCad schematic)
At the start: 3 parts, among them J1 Screw_Terminal_01x02

Commit message: diff circuit
Other:
- sheet HalfBridge_Diff ports: added inen_d; removed none
Changed lines of the file:
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@@
+	)
+	(junction
+		(at 91.44 90.17)
+		(diameter 0)
+		(color 0 0 0 0)
+	)
+	(junction
+		(at 92.71 87.63)
+		(diameter 0)
+		(color 0 0 0 0)
 	)
 	(junction
@@
 	)
 	(junction
+		(at 93.98 85.09)
+		(diameter 0)
+		(color 0 0 0 0)
+	)
+	(junction
 		(at 53.34 95.25)
 		(diameter 0)
@@
 	(wire
 		(pts
-			(xy 87.63 85.09) (xy 99.06 85.09)
+			(xy 87.63 85.09) (xy 93.98 85.09)
 		)
 		(stroke
@@
 	(wire
 		(pts
-			(xy 64.77 60.96) (xy 54.61 60.96)
+			(xy 59.69 60.96) (xy 54.61 60.96)
 		)
 		(stroke
@@
 	(wire
 		(pts
-			(xy 87.63 87.63) (xy 93.98 87.63)
+			(xy 87.63 87.63) (xy 92.71 87.63)
 		)
 		(stroke
@@
 	(wire
 		(pts
-			(xy 64.77 58.42) (xy 53.34 58.42)
+			(xy 59.69 58.42) (xy 53.34 58.42)
 		)
 		(stroke
@@
 	(wire
 		(pts
+			(xy 86.36 63.5) (xy 91.44 63.5)
+		)
+		(stroke
+			(width 0)
+			(type default)
+		)
+	)
+	(wire
+		(pts
 			(xy 91.44 100.33) (xy 102.87 100.33)
 		)
@@
 	(wire
 		(pts
+			(xy 91.44 63.5) (xy 91.44 90.17)
+		)
+		(stroke
+			(width 0)
+			(type default)
+		)
+	)
+	(wire
+		(pts
+			(xy 93.98 85.09) (xy 99.06 85.09)
+		)
+		(stroke
+			(width 0)
+			(type default)
+		)
+	)
+	(wire
+		(pts
 			(xy 53.34 102.87) (xy 102.87 102.87)
 		)
@@
 	(wire
 		(pts
+			(xy 86.36 60.96) (xy 92.71 60.96)
+		)
+		(stroke
+			(width 0)
+			(type default)
+		)
+	)
+	(wire
+		(pts
+			(xy 86.36 58.42) (xy 93.98 58.42)
+		)
+		(stroke
+			(width 0)
+			(type default)
+		)
+	)
+	(wire
+		(pts
 			(xy 142.24 95.25) (xy 154.94 95.25)
 		)
@@
 		(pts
 			(xy 54.61 97.79) (xy 54.61 105.41)
+		)
+		(stroke
+			(width 0)
+			(type default)
+		)
+	)
+	(wire
+		(pts
+			(xy 92.71 60.96) (xy 92.71 87.63)
+		)
+		(stroke
+			(width 0)
+			(type default)
+		)
+	)
+	(wire
+		(pts
+			(xy 92.71 87.63) (xy 93.98 87.63)
+		)
+		(stroke
+			(width 0)
+			(type default)
+		)
+	)
+	(wire
+		(pts
+			(xy 93.98 58.42) (xy 93.98 85.09)
 		)
 		(stroke
@@
 	)
 	(sheet
-		(at 64.77 54.61)
+		(at 59.69 54.61)
 		(size 26.67 10.16)
 		(fields_autoplaced yes)
@@
 		)
 		(property "Sheetname" "HalfBridge_Diff"
-			(at 64.77 53.8984 0)
+			(at 59.69 53.8984 0)
 			(effects
 				(font
@@
 		)
 		(property "Sheetfile" "HalfBridge_Diff.kicad_sch"
-			(at 64.77 65.3546 0)
+			(at 59.69 65.3546 0)
 			(effects
 				(font
@@
 		)
 		(pin "vcc" input
-			(at 64.77 58.42 180)
+			(at 59.69 58.42 180)
 			(effects
 				(font
@@
 		)
 		(pin "gnd" input
-			(at 64.77 60.96 180)
+			(at 59.69 60.96 180)
 			(effects
 				(font
@@
 		)
 		(pin "inb_d" output
-			(at 91.44 60.96 0)
+			(at 86.36 60.96 0)
 			(effects
 				(font
@@
 		)
 		(pin "ina_d" output
-			(at 91.44 58.42 0)
-			(effects
-				(font
+			(at 86.36 58.42 0)
+			(effects
+				(font
+					(size 1.27 1.27)
+				)
+				(justify right)
+			)
+		)
+		(pin "inen_d" output
+			(at 86.36 63.5 0)
+			(effects
+				(font

Commit message: pcb position
Connections:
- net GND is gone; now on net HalfBridge_Diff/gnd: R1.2
Changed lines of the file:
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@@
+	)
+	(junction
+		(at 54.61 105.41)
+		(diameter 0)
+		(color 0 0 0 0)
 	)
 	(junction
@@
 	(wire
 		(pts
+			(xy 54.61 119.38) (xy 54.61 105.41)
+		)
+		(stroke
+			(width 0)
+			(type default)
+		)
+	)
+	(wire
+		(pts
 			(xy 44.45 109.22) (xy 44.45 111.76)
 		)
@@
 		(pts
 			(xy 44.45 95.25) (xy 44.45 101.6)
+		)
+		(stroke
+			(width 0)
+			(type default)
+		)
+	)
+	(wire
+		(pts
+			(xy 44.45 119.38) (xy 54.61 119.38)
 		)
 		(stroke
@@
 					(unit 1)
 				)
-			)
-		)
-	)
-	(symbol
-		(lib_id "power:GND")
-		(at 44.45 119.38 0)
-		(unit 1)
-		(exclude_from_sim no)
-		(in_bom yes)
-		(on_board yes)
-		(dnp no)
-		(fields_autoplaced yes)
-		(property "Reference" "#PWR01"
-			(at 44.45 125.73 0)
-			(effects
-				(font
-					(size 1.27 1.27)
-				)
-				(hide yes)
-			)
-		)
-		(property "Value" "GND"
-			(at 44.45 124.46 0)
-			(effects
-				(font
-					(size 1.27 1.27)
-				)
-			)
-		)
-		(property "Footprint" ""
-			(at 44.45 119.38 0)
-			(effects
-				(font
-					(size 1.27 1.27)
-				)
-				(hide yes)
-			)
-		)
-		(property "Datasheet" ""
-			(at 44.45 119.38 0)
-			(effects
-				(font
-					(size 1.27 1.27)
-				)
-				(hide yes)
-			)
-		)
-		(property "Description" "Power symbol creates a global label with name \"GND\" , ground"
-			(at 44.45 119.38 0)
-			(effects
-				(font
-					(size 1.27 1.27)
-				)
-				(hide yes)
-			)
-		)
-		(pin "1"
-		)
-		(instances
-			(project ""
-				(path "/3c187ffa-7f66-4861-b077-b6965c821fc2"
-					(reference "#PWR01")
-					(unit 1)
-				)
