File: HalfBridge_Optical.kicad_sch (KiCad schematic)
At the start: 12 parts, among them J2 AFBR-2624Z, J3 AFBR-2624Z

Commit message: diff rx
Connections:
- net ina: now also R14.1; no longer R15.1
- net inb: now also R15.1; no longer R14.1
- net vcca: now also C20.1, C21.1, J3.3 (VCCR), L2.1; no longer C17.1, C18.1, J2.3 (VCCR), L1.1
- net vccb: now also C17.1, C18.1, J2.3 (VCCR), L1.1; no longer C20.1, C21.1, J3.3 (VCCR), L2.1
- net xna: now also J3.1 (Data_Out), R14.2; no longer J2.1 (Data_Out), R15.2
- net xnb: now also J2.1 (Data_Out), R15.2; no longer J3.1 (Data_Out), R14.2
Changed lines of the file:
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@@
 		)
 	)
-	(label "xnb"
+	(label "xna"
 		(at 68.58 109.22 0)
 		(fields_autoplaced yes)
@@
 		)
 	)
-	(label "xna"
+	(label "xnb"
 		(at 68.58 73.66 0)
 		(fields_autoplaced yes)
@@
 		)
 	)
-	(label "vcca"
+	(label "vccb"
 		(at 58.42 57.15 0)
 		(fields_autoplaced yes)
@@
 		)
 	)
-	(label "vccb"
+	(label "vcca"
 		(at 58.42 99.06 0)
 		(fields_autoplaced yes)
@@
 		)
 	)
-	(hierarchical_label "ina"
+	(hierarchical_label "inb"
 		(shape output)
 		(at 88.9 73.66 0)
@@
 		)
 	)
-	(hierarchical_label "inb"
+	(hierarchical_label "ina"
 		(shape output)
 		(at 88.9 109.22 0)

Commit message: new optical diff xor
Parts:
- added C20: C, Capacitor_SMD:C_0603_1608Metric_Pad1.08x0.95mm_HandSolder, symbol Device:C
- added C23, C26: C, Capacitor_SMD:C_0805_2012Metric_Pad1.18x1.45mm_HandSolder, symbol Device:C
- added J5: AFBR-2624Z, OptoDevice:Broadcom_AFBR-16xxZ_Vertical, symbol Fiber_Optic:AFBR-2624Z
- added L4: L, Inductor_SMD:L_0603_1608Metric_Pad1.05x0.95mm_HandSolder, symbol Device:L
- added R21: R, Resistor_SMD:R_0603_1608Metric_Pad0.98x0.95mm_HandSolder, symbol Device:R
- J2: footprint OptoDevice:Broadcom_AFBR-16xxZ_Horizontal -> OptoDevice:Broadcom_AFBR-16xxZ_Vertical
- J4: renamed from J3; footprint OptoDevice:Broadcom_AFBR-16xxZ_Horizontal -> OptoDevice:Broadcom_AFBR-16xxZ_Vertical
- renumbered C17 to C18, C20 to C19, C18 to C21, C21 to C22, C19 to C24, C22 to C25, L2 to L3, R15 to R19
Connections:
- net gnd: now also C20.2, C23.2, C26.2, J5.2 (VEER), J5.5 (HP), J5.8 (HP)
- net vcc: now also C26.1, L4.2
- net xna renamed oina
- net xnb renamed oinb
- new net inen: R21.1
- new net oinen: J5.1 (Data_Out), R21.2
- new net vccen: C20.1, C23.1, J5.3 (VCCR), L4.1

Commit message: diff circuit
Parts:
- renumbered C18 to C22, C19 to C23, C20 to C24, C21 to C25, C22 to C26, C23 to C27, C24 to C28, C25 to C29, C26 to C30, J2 to J3, L1 to L2, R14 to R20
Changed lines of the file:
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@@
 		(dnp no)
 		(fields_autoplaced yes)
-		(property "Reference" "C22"
+		(property "Reference" "C26"
 			(at 90.17 95.2499 0)
 			(effects
@@
 			(project "HalfBridge_SiC"
 				(path "/3c187ffa-7f66-4861-b077-b6965c821fc2/6b9f2a3a-4d36-43fe-adee-f56a635b1692"
-					(reference "C22")
+					(reference "C26")
 					(unit 1)
 				)
@@
 		(dnp no)
 		(fields_autoplaced yes)
-		(property "Reference" "L1"
+		(property "Reference" "L2"
 			(at 95.25 48.26 90)
 			(effects
@@
 		(dnp no)
 		(fields_autoplaced yes)
-		(property "Reference" "C24"
+		(property "Reference" "C28"
 			(at 105.41 55.8799 0)
 			(effects
@@
 			(project "HalfBridge_SiC"
 				(path "/3c187ffa-7f66-4861-b077-b6965c821fc2/6b9f2a3a-4d36-43fe-adee-f56a635b1692"
-					(reference "C24")
+					(reference "C28")
 					(unit 1)
 				)
@@
 		(dnp no)
 		(fields_autoplaced yes)
-		(property "Reference" "C26"
+		(property "Reference" "C30"
 			(at 105.41 133.3499 0)
 			(effects
@@
 			(project "HalfBridge_SiC"
 				(path "/3c187ffa-7f66-4861-b077-b6965c821fc2/6b9f2a3a-4d36-43fe-adee-f56a635b1692"
-					(reference "C26")
+					(reference "C30")
 					(unit 1)
 				)
@@
 		(dnp no)
 		(fields_autoplaced yes)
-		(property "Reference" "C21"
+		(property "Reference" "C25"
 			(at 90.17 55.8799 0)
 			(effects
@@
 			(project "HalfBridge_SiC"
 				(path "/3c187ffa-7f66-4861-b077-b6965c821fc2/6b9f2a3a-4d36-43fe-adee-f56a635b1692"
-					(reference "C21")
+					(reference "C25")
 					(unit 1)
 				)
@@
 		(on_board yes)
 		(dnp no)
-		(property "Reference" "R14"
+		(property "Reference" "R20"
 			(at 77.47 102.87 90)
 			(effects
@@
 		(dnp no)
 		(fields_autoplaced yes)
-		(property "Reference" "C20"
+		(property "Reference" "C24"
 			(at 80.01 133.3499 0)
 			(effects
@@
 			(project "HalfBridge_SiC"
 				(path "/3c187ffa-7f66-4861-b077-b6965c821fc2/6b9f2a3a-4d36-43fe-adee-f56a635b1692"
-					(reference "C20")
+					(reference "C24")
 					(unit 1)
 				)
@@
 		(dnp no)
 		(fields_autoplaced yes)
-		(property "Reference" "C18"
+		(property "Reference" "C22"
 			(at 80.01 55.8799 0)
 			(effects
@@
 			(project "HalfBridge_SiC"
 				(path "/3c187ffa-7f66-4861-b077-b6965c821fc2/6b9f2a3a-4d36-43fe-adee-f56a635b1692"
-					(reference "C18")
+					(reference "C22")
 					(unit 1)
 				)
@@
 		(dnp no)
 		(fields_autoplaced yes)
-		(property "Reference" "C25"
+		(property "Reference" "C29"
 			(at 105.41 95.2499 0)
 			(effects
@@
 			(project "HalfBridge_SiC"
 				(path "/3c187ffa-7f66-4861-b077-b6965c821fc2/6b9f2a3a-4d36-43fe-adee-f56a635b1692"
-					(reference "C25")
+					(reference "C29")
 					(unit 1)
 				)
@@
 		(dnp no)
 		(fields_autoplaced yes)
-		(property "Reference" "C23"
+		(property "Reference" "C27"
 			(at 90.17 133.3499 0)
 			(effects
@@
 			(project "HalfBridge_SiC"
 				(path "/3c187ffa-7f66-4861-b077-b6965c821fc2/6b9f2a3a-4d36-43fe-adee-f56a635b1692"
-					(reference "C23")
+					(reference "C27")
 					(unit 1)
 				)
@@
 		(dnp no)
 		(fields_autoplaced yes)
-		(property "Reference" "C19"
+		(property "Reference" "C23"
 			(at 80.01 95.2499 0)
 			(effects
@@
 			(project "HalfBridge_SiC"
 				(path "/3c187ffa-7f66-4861-b077-b6965c821fc2/6b9f2a3a-4d36-43fe-adee-f56a635b1692"
-					(reference "C19")
+					(reference "C23")
 					(unit 1)
 				)
@@
 		(dnp no)
 		(fields_autoplaced yes)
-		(property "Reference" "J2"
+		(property "Reference" "J3"
 			(at 49.53 72.3899 0)
 			(effects
